Commit message: Add URDF for goal detection zed

File: urdf/zed_goal.urdf (robot description, URDF)
Before this commit: robot zed_camera, 4 links, 3 joints
Links:
- removed link zed_fuel_center
- removed link zed_fuel_depth_camera
- removed link zed_fuel_left_camera
- removed link zed_fuel_right_camera
- added link zed_goal_center; visual mesh filename=package://zed_wrapper/urdf/ZED.stl
- added link zed_goal_depth_camera
- added link zed_goal_left_camera; visual cylinder length=.031 radius=0.007
- added link zed_goal_right_camera; visual cylinder length=.031 radius=0.007
Joints:
- removed joint zed_fuel_depth_camera_joint
- removed joint zed_fuel_left_camera_joint
- removed joint zed_fuel_right_camera_joint
- added joint zed_goal_depth_camera_joint: type fixed, parent zed_goal_left_camera, child zed_goal_depth_camera, origin xyz=0 0 0 rpy=-1.5707963267948966 0 -1.5707963267948966
- added joint zed_goal_left_camera_joint: type fixed, parent zed_goal_center, child zed_goal_left_camera, origin xyz=0 0.06 0 rpy=0 0 0
- added joint zed_goal_right_camera_joint: type fixed, parent zed_goal_center, child zed_goal_right_camera, origin xyz=0 -0.06 0 rpy=0 0 0
